Commit message: BALANCED

File: src/cartpole_fuzzy/urdf/cartpole.xacro.urdf (robot description, URDF)
Before this commit: robot cartopole, 6 links, 5 joints
Links:
- link ball: geometry visual sphere radius=0.025
Joints:
- joint cart_to_pole: limit lower=-1.50 upper=1.50 effort=1000.0 velocity=1000.0 -> lower=-1.57 upper=1.57 effort=1000.0 velocity=1000.0

Commit message: plotter and world added

File: src/cartpole_fuzzy/urdf/cartpole.xacro.urdf (robot description, URDF)
Before this commit: robot cartopole, 6 links, 5 joints
Joints:
- joint cart_to_pole: limit lower=-1.57 upper=1.57 effort=1000.0 velocity=1000.0 -> effort=1000.0 velocity=1000.0; type revolute -> continuous

Commit message: controller update

File: src/cartpole_fuzzy/urdf/cartpole.xacro.urdf (robot description, URDF)
Before this commit: robot cartopole, 6 links, 5 joints
Links:
- removed link ball
- added link world
- link cart: geometry collision box size=0.1 0.1 0.04; visual box size=0.1 0.1 0.04
- link leg1: geometry collision cylinder length=0.5 radius=0.02; visual cylinder length=0.5 radius=0.02
- link leg2: geometry collision cylinder length=0.5 radius=0.02; visual cylinder length=0.5 radius=0.02
- link pole: geometry collision cylinder length=0.24 radius=0.005; visual cylinder length=0.24 radius=0.005
- link slideBar: geometry collision box size=0.47 0.05 0.05; visual box size=0.47 0.05 0.05
Joints:
- removed joint pole_to_ball
- added joint world_to_slideBar: type fixed, parent world, child slideBar, origin xyz=0 0 0.5
- joint cart_to_pole: limit effort=1000.0 velocity=1000.0 -> effort=10.0 velocity=10.0; origin xyz=0 0 1.1 -> xyz=0 0.04 0.02 rpy=0 0 0
- joint slider_to_cart: limit lower=-15 upper=15 effort=1000.0 velocity=200 -> lower=-0.235 upper=0.235 effort=1000.0 velocity=10.0; origin xyz=0.0 0.0 0.0 -> xyz=0.0 0.0 0.045
- joint slider_to_leg1: origin xyz=-15.0 0.0 0.5 -> xyz=-0.235 0.0 0.0
- joint slider_to_leg2: origin xyz=15 0.0 0.5 -> xyz=0.235 0.0 0.0
