Commit message: Add cartpole runtime package and controllers configuration

File: src/cartpole_description/urdf/cartpole.urdf.xacro (robot description, xacro)
@@ -126,5 +126,5 @@
     <parent link="slideBar"/>
     <child link="cart"/>
-    <limit effort="1000.0" lower="-0.235" upper="0.235" velocity="10.0"/>
+    <limit effort="1000.0" lower="-5" upper="5" velocity="10.0"/>
     <dynamics damping="0.5" friction="0.5"/>
   </joint>

File: src/cartpole_description/urdf/cartpole_control.xacro (robot description, xacro)
@@ -18,4 +18,5 @@
       <command_interface name="position"/>
       <command_interface name="velocity"/>
+      <command_interface name="effort"/>
       <state_interface name="position"/>
       <state_interface name="velocity"/>

Commit message: Update controller configuration and URDF parameters for effort control

File: src/cartpole_description/urdf/cartpole.urdf.xacro (robot description, xacro)
@@ -126,5 +126,5 @@
     <parent link="slideBar"/>
     <child link="cart"/>
-    <limit effort="1000.0" lower="-5" upper="5" velocity="10.0"/>
+    <limit effort="20.0" lower="-0.235" upper="0.235" velocity="10.0"/>
     <dynamics damping="0.5" friction="0.5"/>
   </joint>
@@ -139,11 +139,10 @@
     <child link="leg2"/>
   </joint>
-  <joint name="cart_to_pole" type="continuous">
-    <parent link="cart"/>
-    <child link="pole"/>
-    <origin xyz="0 0.04 0.02" rpy="0 0 0"/>
-    <axis xyz="0 1 0"/>
-    <dynamics damping="0.01" friction="0.0"/>
-    <limit effort="10.0" velocity="10.0"/>
-  </joint>
+<joint name="cart_to_pole" type="continuous">
+  <parent link="cart"/>
+  <child link="pole"/>
+  <origin xyz="0 0.04 0.02" rpy="3.14159 0 0"/>
+  <axis xyz="0 1 0"/>
+  <dynamics damping="0.01" friction="0.0"/>
+</joint>
 </robot>

File: src/cartpole_description/urdf/cartpole_control.xacro (robot description, xacro)
@@ -21,4 +21,5 @@
       <state_interface name="position"/>
       <state_interface name="velocity"/>
+      <state_interface name="effort"/>
     </joint>
     <!-- Pendulumun encoder verisi için (motor kontrolü yok) -->
@@ -26,4 +27,5 @@
       <state_interface name="position"/>
       <state_interface name="velocity"/>
+      <state_interface name="effort"/>
     </joint>
   </ros2_control>
